File: solarcampi/solarcampi.sch (KiCad schematic (older format))
At the start: 11 parts, among them J1 Conn_02x20_Odd_Even, J2 Vin 12V, Q1 IRLML 2244, Q2 BCR 108 SMD, U1 INA226, U2 ATtiny85-20SU

Commit message: Add fuse, add decoupling caps, set footprints
Parts:
- added C3, C5: 100n, Capacitors_SMD:C_0805_HandSoldering, symbol Device:C
- added C4: 1µF, Capacitors_SMD:C_0805_HandSoldering, symbol Device:C
- added F1: 1A, solarcampi:Fuse_SMD_HASF, symbol Device:Fuse
- C1, C2: footprint (none) -> Capacitors_SMD:C_0805_HandSoldering
- J2: footprint (none) -> Connectors:bornier2
- PS1: renamed from PS?; footprint (none) -> solarcampi:MP1584_buck_module; symbol Converter_DCDC:ITX0503SA -> custom:MP1584ENBB
- Q1: footprint Package_TO_SOT_SMD:SOT-23 -> TO_SOT_Packages_SMD:SOT-23
- Q2: footprint (none) -> TO_SOT_Packages_SMD:SOT-23
- R1: renamed from R?; footprint (none) -> Resistors_SMD:R_0805_HandSoldering
- U1: footprint Package_SO:MSOP-10_3x3mm_P0.5mm -> Housings_SSOP:MSOP-10_3x3mm_Pitch0.5mm
- U2: footprint Package_SO:SOIJ-8_5.3x5.3mm_P1.27mm -> Housings_SOIC:SOIJ-8_5.3x5.3mm_Pitch1.27mm
- U3: renamed from U?; footprint Package_TO_SOT_SMD:SOT-353_SC-70-5 -> TO_SOT_Packages_SMD:SOT-353_SC-70-5_Handsoldering
Connections:
- net +12V: now also C3.1, F1.1; no longer J2.2 (Pin_2)
- net +3V3: now also C4.1, C5.1
- net GND: now also PS1.2 (VINGND), PS1.3 (VOUTGND), C3.2, C4.2, C5.2; no longer PS1.1 (-Vin), PS1.7 (-Vout)
- net at J1.2 (Pin_2): now also PS1.4 (VOUT); no longer PS1.6 (+Vout)
- net +12VA: now reaches Q1.3 (D)
- net +12VA: now also PS1.1 (VIN); no longer PS1.2 (+Vin)
- new net: F1.2, J2.2 (Pin_2)
- no-connect marks 2 -> 43
Other:
- moved on the sheet: C1, U3

Commit message: Add ISP header, FTDI header, more caps, power switching for INA and 2 I2C busses
Parts:
- removed C2: 100n, Capacitors_SMD:C_0805_HandSoldering, symbol Device:C
- removed U2: ATtiny85-20SU, Housings_SOIC:SOIJ-8_5.3x5.3mm_Pitch1.27mm, symbol MCU_Microchip_ATtiny:ATtiny85-20SU
- added C2: 100n, Capacitor_SMD:C_0805_2012Metric_Pad1.15x1.40mm_HandSolder, symbol solarcampi-rescue:C-Device
- added C6: 100n, Capacitor_SMD:C_0805_2012Metric_Pad1.15x1.40mm_HandSolder, symbol Device:C
- added C7, C8: 10µ, Capacitor_SMD:C_0805_2012Metric_Pad1.15x1.40mm_HandSolder, symbol Device:C
- added J3: AVR-ISP-6, Connector_IDC:IDC-Header_2x03_P2.54mm_Vertical, symbol Connector:AVR-ISP-6
- added J4: FTDI, Connector_PinHeader_2.54mm:PinHeader_1x06_P2.54mm_Vertical, symbol Connector:Conn_01x06_Male
- added JP1: Jumper_2_Open, Jumper:SolderJumper-2_P1.3mm_Open_Pad1.0x1.5mm, symbol Jumper:Jumper_2_Open
- added R2: 10k, Resistor_SMD:R_0805_2012Metric_Pad1.15x1.40mm_HandSolder, symbol Device:R
- added R3, R4: 4k7, Resistor_SMD:R_0805_2012Metric_Pad1.15x1.40mm_HandSolder, symbol Device:R
- added U2: ATmega328P-AU, Package_QFP:TQFP-32_7x7mm_P0.8mm, symbol MCU_Microchip_ATmega:ATmega328P-AU
- C1, C3, C4, C5: footprint Capacitors_SMD:C_0805_HandSoldering -> Capacitor_SMD:C_0805_2012Metric_Pad1.15x1.40mm_HandSolder; symbol Device:C -> solarcampi-rescue:C-Device
- F1: symbol Device:Fuse -> solarcampi-rescue:Fuse-Device
- J1: symbol Connector_Generic:Conn_02x20_Odd_Even -> solarcampi-rescue:Conn_02x20_Odd_Even-Connector_Generic
- J2: footprint Connectors:bornier2 -> TerminalBlock:TerminalBlock_bornier-2_P5.08mm; symbol Connector:Screw_Terminal_01x02 -> solarcampi-rescue:Screw_Terminal_01x02-Connector
- Q1: footprint TO_SOT_Packages_SMD:SOT-23 -> Package_TO_SOT_SMD:SOT-23; symbol Transistor_FET:IRLML6402 -> solarcampi-rescue:IRLML6402-Transistor_FET
- Q2: footprint TO_SOT_Packages_SMD:SOT-23 -> Package_TO_SOT_SMD:SOT-23; symbol Transistor_BJT:DTC123J -> solarcampi-rescue:DTC123J-Transistor_BJT
- R1: footprint Resistors_SMD:R_0805_HandSoldering -> Resistor_SMD:R_0805_2012Metric_Pad1.15x1.40mm_HandSolder; symbol Device:R -> solarcampi-rescue:R-Device
- U1: footprint Housings_SSOP:MSOP-10_3x3mm_Pitch0.5mm -> Package_SO:MSOP-10_3x3mm_P0.5mm; symbol Analog_ADC:INA226 -> solarcampi-rescue:INA226-Analog_ADC
- U3: footprint TO_SOT_Packages_SMD:SOT-353_SC-70-5_Handsoldering -> Package_TO_SOT_SMD:SOT-353_SC-70-5_Handsoldering; symbol Regulator_Linear:TPS71533__SC70 -> solarcampi-rescue:TPS71533__SC70-Regulator_Linear
Connections:
- net +3V3: now also C2.1, C7.1, JP1.1 (A), R2.1, U2.18 (AVCC), U2.4 (VCC), U2.6 (VCC); no longer C5.1, U1.6 (Vs)
- net GND: now also C2.2, C6.2, C7.2, C8.2, J3.6 (GND), J4.1 (Pin_1), U2.21 (GND), U2.3 (GND), U2.5 (GND)
- net TX: now reaches J1.10 (Pin_10)
- net TX: now also J4.4 (Pin_4)
- net at J1.2 (Pin_2), PS1.4 (VOUT): now also C8.1
- net RPI_SDA: now reaches J1.3 (Pin_3)
- net RPI_SDA: now also U2.27 (PC4)
- net RPI_SCL: now reaches J1.5 (Pin_5)
- net RPI_SCL: now also U2.28 (PC5)
- net RPI_SHDN: now reaches J1.7 (Pin_7)
- net RPI_SHDN: now also U2.32 (PD2)
- net RX: now reaches J1.8 (Pin_8)
- net RX: now also J4.5 (Pin_5)
- net AVR_SDA: now reaches U1.4 (SDA)
- net AVR_SDA: now also R4.1, U2.1 (PD3)
- net AVR_SCL: now reaches U1.5 (SCL)
- net AVR_SCL: now also R3.1, U2.2 (PD4)
- net at Q2.1 (B): now also U2.11 (PD7)
- new net: J3.2 (VCC), JP1.2 (B)
- new net AVR_I2C_PULLUP: R3.2, R4.2, U2.9 (PD5)
- new net INA_3V3: C5.1, U1.6 (Vs), U2.10 (PD6)
- new net MISO: J3.1 (MISO), U2.16 (PB4)
- new net MOSI: J3.4 (MOSI), U2.15 (PB3)
- new net SCK: J3.3 (SCK), U2.17 (PB5)
- new net ~RST: C6.1, J3.5 (~RST), R2.2, U2.29 (~RESET~/PC6)
- no-connect marks 43 -> 39
Other:
- moved on the sheet: C5, U1

Commit message: Component placement v1
Connections:
- net AVR_I2C_PULLUP: now also U2.19 (ADC6); no longer U2.9 (PD5)
- net AVR_SCL: now also R4.1, U2.23 (PC0); no longer R3.1, U2.2 (PD4)
- net AVR_SDA: now also R3.1, U2.24 (PC1); no longer R4.1, U2.1 (PD3)
Other:
- moved on the sheet: C2, C7, R3, R4
Changed lines of the file:
@@
 L solarcampi-rescue:C-Device C2
 U 1 1 5CF4ECCB
-P 3050 1350
-F 0 "C2" H 3165 1396 50  0000 L CNN
-F 1 "100n" H 3165 1305 50  0000 L CNN
-F 2 "Capacitor_SMD:C_0805_2012Metric_Pad1.15x1.40mm_HandSolder" H 3088 1200 50  0001 C CNN
-F 3 "~" H 3050 1350 50  0001 C CNN
-	1    3050 1350
+P 2650 900
+F 0 "C2" H 2765 946 50  0000 L CNN
+F 1 "100n" H 2765 855 50  0000 L CNN
+F 2 "Capacitor_SMD:C_0805_2012Metric_Pad1.15x1.40mm_HandSolder" H 2688 750 50  0001 C CNN
+F 3 "~" H 2650 900 50  0001 C CNN
+	1    2650 900
 	1    0    0    -1
 $EndComp
@@
 L solarcampi-rescue:+3V3-power #PWR01
 U 1 1 5CF4ECD1
-P 3050 1200
-F 0 "#PWR01" H 3050 1050 50  0001 C CNN
-F 1 "+3V3" H 3065 1373 50  0000 C CNN
-F 2 "" H 3050 1200 50  0001 C CNN
-F 3 "" H 3050 1200 50  0001 C CNN
-	1    3050 1200
+P 2650 750
+F 0 "#PWR01" H 2650 600 50  0001 C CNN
+F 1 "+3V3" H 2665 923 50  0000 C CNN
+F 2 "" H 2650 750 50  0001 C CNN
+F 3 "" H 2650 750 50  0001 C CNN
+	1    2650 750
 	1    0    0    -1
 $EndComp
@@
 L solarcampi-rescue:GND-power #PWR02
 U 1 1 5CF4ECD7
-P 3050 1500
-F 0 "#PWR02" H 3050 1250 50  0001 C CNN
-F 1 "GND" H 3055 1327 50  0000 C CNN
-F 2 "" H 3050 1500 50  0001 C CNN
-F 3 "" H 3050 1500 50  0001 C CNN
-	1    3050 1500
+P 2650 1050
+F 0 "#PWR02" H 2650 800 50  0001 C CNN
+F 1 "GND" H 2655 877 50  0000 C CNN
+F 2 "" H 2650 1050 50  0001 C CNN
+F 3 "" H 2650 1050 50  0001 C CNN
+	1    2650 1050
 	1    0    0    -1
 $EndComp
@@
 Text Label 4650 2900 0    50   ~ 0
 RPI_SHDN
-Text Label 4900 3000 0    50   ~ 0
+Text Label 4900 2000 0    50   ~ 0
 AVR_SDA
-Text Label 4900 3100 0    50   ~ 0
+Text Label 4900 1900 0    50   ~ 0
 AVR_SCL
 Text Label 1950 3900 0    50   ~ 0
@@
 L Device:R R3
 U 1 1 5D013A55
-P 5200 3250
-F 0 "R3" H 5270 3296 50  0000 L CNN
-F 1 "4k7" H 5270 3205 50  0000 L CNN
-F 2 "Resistor_SMD:R_0805_2012Metric_Pad1.15x1.40mm_HandSolder" V 5130 3250 50  0001 C CNN
-F 3 "~" H 5200 3250 50  0001 C CNN
-	1    5200 3250
+P 5200 2150
+F 0 "R3" H 5270 2196 50  0000 L CNN
+F 1 "4k7" H 5270 2105 50  0000 L CNN
+F 2 "Resistor_SMD:R_0805_2012Metric_Pad1.15x1.40mm_HandSolder" V 5130 2150 50  0001 C CNN
+F 3 "~" H 5200 2150 50  0001 C CNN
+	1    5200 2150
 	1    0    0    -1
 $EndComp
@@
 L Device:R R4
 U 1 1 5D01456F
-P 5450 3150
-F 0 "R4" H 5520 3196 50  0000 L CNN
-F 1 "4k7" H 5520 3105 50  0000 L CNN
-F 2 "Resistor_SMD:R_0805_2012Metric_Pad1.15x1.40mm_HandSolder" V 5380 3150 50  0001 C CNN
-F 3 "~" H 5450 3150 50  0001 C CNN
-	1    5450 3150
-	1    0    0    -1
-$EndComp
-Wire Wire Line
-	4650 3100 5200 3100
-Wire Wire Line
-	4650 3000 5450 3000
-Wire Wire Line
-	5200 3400 5450 3400
-Wire Wire Line
-	5450 3400 5450 3300
-Wire Wire Line
-	5200 3400 4950 3400
+P 5450 2050
+F 0 "R4" H 5520 2096 50  0000 L CNN
+F 1 "4k7" H 5520 2005 50  0000 L CNN
+F 2 "Resistor_SMD:R_0805_2012Metric_Pad1.15x1.40mm_HandSolder" V 5380 2050 50  0001 C CNN
+F 3 "~" H 5450 2050 50  0001 C CNN
+	1    5450 2050
+	1    0    0    -1
+$EndComp
+Wire Wire Line
+	4650 2000 5200 2000
+Wire Wire Line
+	4650 1900 5450 1900
+Wire Wire Line
+	5450 2300 5450 2200
 Wire Wire Line
 	4950 3400 4950 3200
 Wire Wire Line
 	4950 3200 4650 3200
-Connection ~ 5200 3400
-Text Label 5450 3400 0    50   ~ 0
+Text Label 5450 2300 0    50   ~ 0
 AVR_I2C_PULLUP
 Text Label 1550 3400 0    50   ~ 0
@@
 L Device:C C7
 U 1 1 5D096BE4
-P 2650 1350
-F 0 "C7" H 2765 1396 50  0000 L CNN
-F 1 "10µ" H 2765 1305 50  0000 L CNN
-F 2 "Capacitor_SMD:C_0805_2012Metric_Pad1.15x1.40mm_HandSolder" H 2688 1200 50  0001 C CNN
-F 3 "~" H 2650 1350 50  0001 C CNN
-	1    2650 1350
-	1    0    0    -1
-$EndComp
-Connection ~ 3050 1200
-Connection ~ 3050 1500
-Wire Wire Line
-	2650 1200 3050 1200
-Wire Wire Line
-	2650 1500 3050 1500
+P 2250 900
+F 0 "C7" H 2365 946 50  0000 L CNN
+F 1 "10µ" H 2365 855 50  0000 L CNN
+F 2 "Capacitor_SMD:C_0805_2012Metric_Pad1.15x1.40mm_HandSolder" H 2288 750 50  0001 C CNN
+F 3 "~" H 2250 900 50  0001 C CNN
+	1    2250 900
+	1    0    0    -1
+$EndComp
+Connection ~ 2650 750
+Connection ~ 2650 1050
+Wire Wire Line
+	2250 750  2650 750
+Wire Wire Line
+	2250 1050 2650 1050
 Connection ~ 10600 2000
 $Comp
@@
 	1    0    0    -1
 $EndComp
+Wire Wire Line
+	5200 2300 5450 2300
+Text Label 3450 1200 2    50   ~ 0
+AVR_I2C_PULLUP
 $EndSCHEMATC

Commit message: Route everything
Parts:
- added C9: 100n, Capacitor_SMD:C_0805_2012Metric_Pad1.15x1.40mm_HandSolder, symbol Device:C
Connections:
- net AVR_I2C_PULLUP: now also C9.1
- net AVR_SCL: now also R3.1, U2.22 (ADC7); no longer R4.1, U2.23 (PC0)
- net AVR_SDA: now also R4.1, U2.23 (PC0); no longer R3.1, U2.24 (PC1)
- net GND: now also C9.2
- net INA_3V3: now also U2.24 (PC1); no longer U2.10 (PD6)
- net RPI_5V: now reaches C8.1, J1.2 (Pin_2), PS1.4 (VOUT)
- net AVR_PWR_EN: now reaches Q2.1 (B), U2.11 (PD7)
- net +12VA renamed +12V_SWITCHED
Other:
- moved on the sheet: R3
Changed lines of the file:
@@
 	6550 2000 6550 2050
 Connection ~ 6550 2050
-$Comp
-L solarcampi-rescue:+12VA-power #PWR0120
-U 1 1 5CF5E1D1
-P 7400 2000
-F 0 "#PWR0120" H 7400 1850 50  0001 C CNN
-F 1 "+12VA" H 7415 2173 50  0000 C CNN
-F 2 "" H 7400 2000 50  0001 C CNN
-F 3 "" H 7400 2000 50  0001 C CNN
-	1    7400 2000
-	1    0    0    -1
-$EndComp
 Wire Wire Line
 	1700 950  1750 950
@@
 Connection ~ 1700 1250
 Wire Wire Line
-	7150 2050 7400 2050
-Wire Wire Line
-	7400 2000 7400 2050
-Wire Wire Line
 	10600 1700 8750 1700
 Wire Wire Line
 	8750 1700 8750 2050
-Wire Wire Line
-	7400 2050 7550 2050
-Connection ~ 7400 2050
 $Comp
 L Connector:Conn_01x06_Male J4
@@
 Text Label 4650 2900 0    50   ~ 0
 RPI_SHDN
-Text Label 4900 2000 0    50   ~ 0
+Text Label 5100 1900 2    50   ~ 0
 AVR_SDA
-Text Label 4900 1900 0    50   ~ 0
+Text Label 3050 1300 0    50   ~ 0
 AVR_SCL
 Text Label 1950 3900 0    50   ~ 0
@@
 L Device:R R3
 U 1 1 5D013A55
-P 5200 2150
-F 0 "R3" H 5270 2196 50  0000 L CNN
-F 1 "4k7" H 5270 2105 50  0000 L CNN
-F 2 "Resistor_SMD:R_0805_2012Metric_Pad1.15x1.40mm_HandSolder" V 5130 2150 50  0001 C CNN
-F 3 "~" H 5200 2150 50  0001 C CNN
-	1    5200 2150
-	1    0    0    -1
+P 2900 1450
+F 0 "R3" H 2970 1496 50  0000 L CNN
+F 1 "4k7" H 2970 1405 50  0000 L CNN
+F 2 "Resistor_SMD:R_0805_2012Metric_Pad1.15x1.40mm_HandSolder" V 2830 1450 50  0001 C CNN
+F 3 "~" H 2900 1450 50  0001 C CNN
+	1    2900 1450
+	-1   0    0    -1
 $EndComp
 $Comp
@@
 $EndComp
 Wire Wire Line
-	4650 2000 5200 2000
+	3450 1300 2900 1300
 Wire Wire Line
 	4650 1900 5450 1900
-Wire Wire Line
-	5450 2300 5450 2200
 Wire Wire Line
 	4950 3400 4950 3200
@@
 Text Label 650  3650 0    50   ~ 0
 INA_3V3
-Text Label 4650 3300 0    50   ~ 0
+Text Label 4750 2000 0    50   ~ 0
 INA_3V3
 Wire Wire Line
@@
 	1    0    0    -1
 $EndComp
-Wire Wire Line
-	5200 2300 5450 2300
 Text Label 3450 1200 2    50   ~ 0
 AVR_I2C_PULLUP
+Text Label 2900 1600 3    50   ~ 0
+AVR_I2C_PULLUP
+Wire Wire Line
+	5450 2200 5450 2300
+Wire Wire Line
+	4650 2000 4750 2000
+$Comp
+L Device:C C9
+U 1 1 5D17957D
+P 2700 2650
+F 0 "C9" H 2815 2696 50  0000 L CNN
+F 1 "100n" H 2815 2605 50  0000 L CNN
+F 2 "Capacitor_SMD:C_0805_2012Metric_Pad1.15x1.40mm_HandSolder" H 2738 2500 50  0001 C CNN
+F 3 "~" H 2700 2650 50  0001 C CNN
+	1    2700 2650
+	1    0    0    -1
+$EndComp
+Text Label 2700 2500 0    50   ~ 0
+AVR_I2C_PULLUP
+$Comp
+L power:GND #PWR05
+U 1 1 5D17E891
+P 2700 2800
+F 0 "#PWR05" H 2700 2550 50  0001 C CNN
+F 1 "GND" H 2705 2627 50  0000 C CNN
+F 2 "" H 2700 2800 50  0001 C CNN
+F 3 "" H 2700 2800 50  0001 C CNN
+	1    2700 2800
+	1    0    0    -1
+$EndComp
+Text Label 8900 1700 0    50   ~ 0
+RPI_5V
+Wire Wire Line
+	7150 2050 7550 2050
+Text Label 7350 2050 1    50   ~ 0
++12V_SWITCHED
+Text Label 5600 3500 0    50   ~ 0
+AVR_PWR_EN
 $EndSCHEMATC
