File: pcb/_autosave-solarcampi.kicad_pcb (KiCad board)
At the start: 2 copper layers, 65 x 30 mm, 30 parts, among them J2 Vin 12V, J3 AVR-ISP-6, Q1 IRLML 2244, Q2 BCR 108 SMD, U1 INA226, U2 ATmega328P-AU, U3 TPS71533__SC70

Commit message: Schematic RevB
Parts:
- removed C3: 100n, Capacitor_SMD:C_0805_2012Metric_Pad1.15x1.40mm_HandSolder
- removed C4: 1µF, Capacitor_SMD:C_0805_2012Metric_Pad1.15x1.40mm_HandSolder
- removed U3: TPS71533__SC70, Package_TO_SOT_SMD:SOT-353_SC-70-5_Handsoldering
Routing:
- net +3V3: track 67.0 -> 29.1 mm
- net +12V: track 63.7 -> 33.8 mm, vias 3 -> 2
