File: pcb/solarcampi.kicad_pcb (KiCad board)
At the start: 2 copper layers, 65 x 30 mm, 46 parts, among them J1 Vin 12V, J2 AVR-ISP-6, J3 FTDI_AVR, J4 Conn_02x20_Odd_Even, J5 FTDI_RPI, Q1 Q_NMOS_GDS, Q2 IRLML 2244, Q3 Q_NMOS_GDS, Q4 Q_NMOS_GDS, U1 INA226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

Commit message: Add PCB-art
Parts:
- added G***: LOGO, solarcampi:catboy, B.Cu at (59.6, 66.1)
