File: pcb/solarcampi.sch (KiCad schematic (older format))
At the start: 50 parts, among them J1 Vin 12V, J2 AVR-ISP-6, J3 FTDI_AVR, J4 Conn_02x20_Odd_Even, J5 FTDI_RPI, J6 Shunt, Q1 Q_NMOS_GSD, Q2 IRLML 2244, Q3 Q_NMOS_GSD, Q4 Q_NMOS_GSD, U1 INA226, U2 TPS71533__SC70, U3 ATmega328P-AU

Commit message: Finishing touches on RevC
Parts:
- C10: value 100u -> 100µ
- C12: value C -> 100n
- C13: renamed from C?; value CP -> 33µ
- C6: value C -> 22µ
- D3: value D_Zener -> 5.6V
- F2: value Fuse -> 1A
- JP2: value Jumper_NO_Small -> Enable RPi
- JP3, JP4, JP5: value Jumper_NO_Small -> NC
- Q1, Q3, Q4: value Q_NMOS_GSD -> 2N7002
- Q2: value IRLML 2244 -> DMP3099L
- R11: value R -> .02R
- R2: value R -> 100k
Other:
- moved on the sheet: C12, J6, R11
Changed lines of the file:
@@
 Sheet 1 1
 Title "Solar Camera Pi"
-Date "2019-05-27"
-Rev "A"
+Date "2019-07-27"
+Rev "C"
 Comp "Tobias Mädel (@manawyrm), Tobias Schramm (@Toble_Miner)"
 Comment1 "https://tbspace.de"
@@
 P 6950 2150
 F 0 "Q2" V 7293 2150 50  0000 C CNN
-F 1 "IRLML 2244" V 7202 2150 50  0000 C CNN
+F 1 "DMP3099L" V 7202 2150 50  0000 C CNN
 F 2 "Package_TO_SOT_SMD:SOT-23" H 7150 2075 50  0001 L CIN
-F 3 "https://www.infineon.com/dgdl/irlml6402pbf.pdf?fileId=5546d462533600a401535668d5c2263c" H 6950 2150 50  0001 L CNN
+F 3 "https://www.mouser.de/datasheet/2/115/DMP3099L-266220.pdf" H 6950 2150 50  0001 L CNN
 	1    6950 2150
 	0    1    -1   0
@@
 P 8900 2700
 F 0 "JP3" H 8900 2885 50  0000 C CNN
-F 1 "Jumper_NO_Small" H 8900 2794 50  0000 C CNN
+F 1 "NC" H 8900 2794 50  0000 C CNN
 F 2 "Jumper:SolderJumper-2_P1.3mm_Bridged_Pad1.0x1.5mm" H 8900 2700 50  0001 C CNN
 F 3 "~" H 8900 2700 50  0001 C CNN
@@
 P 8900 3000
 F 0 "JP4" H 8900 3185 50  0000 C CNN
-F 1 "Jumper_NO_Small" H 8900 3094 50  0000 C CNN
+F 1 "NC" H 8900 3094 50  0000 C BNN
 F 2 "Jumper:SolderJumper-2_P1.3mm_Bridged_Pad1.0x1.5mm" H 8900 3000 50  0001 C CNN
 F 3 "~" H 8900 3000 50  0001 C CNN
 	1    8900 3000
-	1    0    0    -1
-$EndComp
-$Comp
-L Device:Jumper_NC_Small JP5
-U 1 1 5D09C8F7
-P 8900 3300
-F 0 "JP5" H 8900 3485 50  0000 C CNN
-F 1 "Jumper_NO_Small" H 8900 3394 50  0000 C CNN
-F 2 "Jumper:SolderJumper-2_P1.3mm_Bridged_Pad1.0x1.5mm" H 8900 3300 50  0001 C CNN
-F 3 "~" H 8900 3300 50  0001 C CNN
-	1    8900 3300
 	1    0    0    -1
 $EndComp
@@
 P 9600 1700
 F 0 "F2" V 9403 1700 50  0000 C CNN
-F 1 "Fuse" V 9494 1700 50  0000 C CNN
+F 1 "1A" V 9494 1700 50  0000 C CNN
 F 2 "Fuse:Fuse_0805_2012Metric_Pad1.15x1.40mm_HandSolder" V 9530 1700 50  0001 C CNN
 F 3 "~" H 9600 1700 50  0001 C CNN
@@
 P 10950 1900
 F 0 "D3" V 10904 1979 50  0000 L CNN
-F 1 "D_Zener" V 10995 1979 50  0000 L CNN
+F 1 "5.6V" V 10995 1979 50  0000 L CNN
 F 2 "Diode_SMD:D_SOD-123" H 10950 1900 50  0001 C CNN
 F 3 "~" H 10950 1900 50  0001 C CNN
@@
 P 5300 3750
 F 0 "R2" H 5370 3796 50  0000 L CNN
-F 1 "R" H 5370 3705 50  0000 L CNN
+F 1 "100k" H 5370 3705 50  0000 L CNN
 F 2 "Resistor_SMD:R_0805_2012Metric_Pad1.15x1.40mm_HandSolder" V 5230 3750 50  0001 C CNN
 F 3 "~" H 5300 3750 50  0001 C CNN
@@
 P 6850 1250
 F 0 "C6" H 6735 1204 50  0000 R CNN
-F 1 "C" H 6735 1295 50  0000 R CNN
+F 1 "22µ" H 6735 1295 50  0000 R CNN
 F 2 "Capacitor_SMD:C_0805_2012Metric_Pad1.15x1.40mm_HandSolder" H 6888 1100 50  0001 C CNN
 F 3 "~" H 6850 1250 50  0001 C CNN
@@
 P 6150 2850
 F 0 "JP2" H 6150 3035 50  0000 C CNN
-F 1 "Jumper_NO_Small" H 6150 2944 50  0000 C CNN
+F 1 "Enable RPi" H 6150 2944 50  0000 C CNN
 F 2 "Connector_PinHeader_2.54mm:PinHeader_1x02_P2.54mm_Vertical" H 6150 2850 50  0001 C CNN
 F 3 "~" H 6150 2850 50  0001 C CNN
@@
 P 6850 3200
 F 0 "Q1" H 6700 3250 50  0000 L CNN
-F 1 "Q_NMOS_GSD" H 6300 3350 50  0000 L CNN
+F 1 "2N7002" H 6500 3350 50  0000 L CNN
 F 2 "Package_TO_SOT_SMD:SOT-23" H 7050 3300 50  0001 C CNN
 F 3 "~" H 6850 3200 50  0001 C CNN
@@
 P 7300 3200
 F 0 "Q3" H 7150 3250 50  0000 L CNN
-F 1 "Q_NMOS_GSD" H 6750 3350 50  0000 L CNN
+F 1 "2N7002" H 6950 3350 50  0000 L CNN
 F 2 "Package_TO_SOT_SMD:SOT-23" H 7500 3300 50  0001 C CNN
 F 3 "~" H 7300 3200 50  0001 C CNN
@@
 P 9250 4200
 F 0 "Q4" H 9456 4246 50  0000 L CNN
-F 1 "Q_NMOS_GSD" H 9456 4155 50  0000 L CNN
+F 1 "2N7002" H 9456 4155 50  0000 L CNN
 F 2 "Package_TO_SOT_SMD:SOT-23" H 9450 4300 50  0001 C CNN
 F 3 "~" H 9250 4200 50  0001 C CNN
@@
 P 2700 1900
 F 0 "C10" V 2550 1900 50  0000 C CNN
-F 1 "100u" V 2450 1900 50  0000 C CNN
+F 1 "100µ" V 2450 1900 50  0000 C CNN
 F 2 "Capacitor_SMD:C_1210_3225Metric_Pad1.42x2.65mm_HandSolder" H 2738 1750 50  0001 C CNN
 F 3 "~" H 2700 1900 50  0001 C CNN
@@
 	1    0    0    -1
 $EndComp
-Text Label 1250 4200 0    50   ~ 0
+Text Label 1200 4200 0    50   ~ 0
 SHUNT+
-Text Label 1250 4600 0    50   ~ 0
+Text Label 1200 4600 0    50   ~ 0
 SHUNT-
 Wire Wire Line
@@
 L Device:C C12
 U 1 1 5D49A050
-P 1600 4400
-F 0 "C12" H 1715 4446 50  0000 L CNN
-F 1 "C" H 1715 4355 50  0000 L CNN
-F 2 "Capacitor_SMD:C_0805_2012Metric_Pad1.15x1.40mm_HandSolder" H 1638 4250 50  0001 C CNN
-F 3 "~" H 1600 4400 50  0001 C CNN
-	1    1600 4400
+P 1550 4400
+F 0 "C12" H 1665 4446 50  0000 L CNN
+F 1 "100n" H 1665 4355 50  0000 L CNN
+F 2 "Capacitor_SMD:C_0805_2012Metric_Pad1.15x1.40mm_HandSolder" H 1588 4250 50  0001 C CNN
+F 3 "~" H 1550 4400 50  0001 C CNN
+	1    1550 4400
 	1    0    0    -1
 $EndComp
@@
 L Device:R R11
 U 1 1 5D4BFA64
-P 1250 4400
-F 0 "R11" H 1320 4446 50  0000 L CNN
-F 1 "R" H 1320 4355 50  0000 L CNN
-F 2 "Resistor_SMD:R_1210_3225Metric_Pad1.42x2.65mm_HandSolder" V 1180 4400 50  0001 C CNN
-F 3 "~" H 1250 4400 50  0001 C CNN
-	1    1250 4400
+P 1200 4400
+F 0 "R11" H 1270 4446 50  0000 L CNN
+F 1 ".02R" H 1270 4355 50  0000 L CNN
+F 2 "Resistor_SMD:R_1210_3225Metric_Pad1.42x2.65mm_HandSolder" V 1130 4400 50  0001 C CNN
+F 3 "~" H 1200 4400 50  0001 C CNN
+	1    1200 4400
 	1    0    0    -1
 $EndComp
@@
 	1900 4450 1900 4600
 Wire Wire Line
-	1600 4250 1600 4200
-Connection ~ 1600 4200
-Wire Wire Line
-	1600 4200 1900 4200
-Wire Wire Line
-	1600 4550 1600 4600
-Connection ~ 1600 4600
-Wire Wire Line
-	1600 4600 1900 4600
-Wire Wire Line
-	1250 4250 1250 4200
-Wire Wire Line
-	1250 4200 1600 4200
-Wire Wire Line
-	1250 4550 1250 4600
-Wire Wire Line
-	1250 4600 1600 4600
-Wire Wire Line
-	1100 4350 1100 4200
-Wire Wire Line
-	1100 4200 1250 4200
-Connection ~ 1250 4200
-Wire Wire Line
-	1100 4450 1100 4600
-Wire Wire Line
-	1100 4600 1250 4600
-Connection ~ 1250 4600
+	1550 4250 1550 4200
+Connection ~ 1550 4200
+Wire Wire Line
+	1550 4550 1550 4600
+Connection ~ 1550 4600
+Wire Wire Line
+	1200 4250 1200 4200
+Wire Wire Line
+	1200 4200 1550 4200
+Wire Wire Line
+	1200 4550 1200 4600
+Wire Wire Line
+	1200 4600 1550 4600
+Wire Wire Line
+	1050 4350 1050 4200
+Wire Wire Line
+	1050 4200 1200 4200
+Connection ~ 1200 4200
+Wire Wire Line
+	1050 4450 1050 4600
+Wire Wire Line
+	1050 4600 1200 4600
+Connection ~ 1200 4600
 $Comp
 L solarcampi-rescue:Screw_Terminal_01x02-Connector J6
 U 1 1 5D510791
-P 900 4350
-F 0 "J6" H 980 4342 50  0000 L CNN
-F 1 "Shunt" H 980 4251 50  0000 L CNN
-F 2 "solarcampi:TerminalBlock_bornier-2_P5.08mm" H 900 4350 50  0001 C CNN
-F 3 "~" H 900 4350 50  0001 C CNN
-	1    900  4350
+P 850 4350
+F 0 "J6" H 930 4342 50  0000 L CNN
+F 1 "Shunt" H 930 4251 50  0000 L CNN
+F 2 "solarcampi:TerminalBlock_bornier-2_P5.08mm" H 850 4350 50  0001 C CNN
+F 3 "~" H 850 4350 50  0001 C CNN
+	1    850  4350
 	-1   0    0    -1
 $EndComp
@@
 $EndComp
 $Comp
-L Device:CP C?
+L Device:CP C13
 U 1 1 5D5BD9B1
 P 2250 1750
-F 0 "C?" H 2368 1796 50  0000 L CNN
-F 1 "CP" H 2368 1705 50  0000 L CNN
+F 0 "C13" H 2368 1796 50  0000 L CNN
+F 1 "33µ" H 2368 1705 50  0000 L CNN
 F 2 "Capacitor_SMD:CP_Elec_5x5.4" H 2288 1600 50  0001 C CNN
 F 3 "~" H 2250 1750 50  0001 C CNN
@@
 	2550 1900 2250 1900
 Connection ~ 2250 1900
+Wire Wire Line
+	1550 4200 1900 4200
+Wire Wire Line
+	1550 4600 1900 4600
+$Comp
+L Device:Jumper_NC_Small JP5
+U 1 1 5D09C8F7
+P 8900 3300
+F 0 "JP5" H 8900 3485 50  0000 C CNN
+F 1 "NC" H 8900 3394 50  0000 C CNN
+F 2 "Jumper:SolderJumper-2_P1.3mm_Bridged_Pad1.0x1.5mm" H 8900 3300 50  0001 C CNN
+F 3 "~" H 8900 3300 50  0001 C CNN
+	1    8900 3300
+	1    0    0    -1
+$EndComp
 $EndSCHEMATC
